File: LBriduino.brd (EAGLE design)
At the start: 45.4 x 27.9 mm, 13 parts, among them J1 105017-0001

Commit message: reverted BM019 input to VIN
Connections:
- new net N$5: BM2.SS0, BM2.VDD
- net SWITCH: now also BM2.VIN; no longer BM2.SS0, BM2.VDD
Routing:
- net N$5: track 0.00 -> 2.71 mm
- net SWITCH: track 48.5 -> 49.9 mm
Changed lines of the file:
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@@
 <setting verticaltext="up"/>
 </settings>
-<grid distance="50" unitdist="mil" unit="inch" style="lines" multiple="1" display="yes" altdistance="0.005" altunitdist="inch" altunit="inch"/>
+<grid distance="50" unitdist="mil" unit="inch" style="lines" multiple="1" display="no" altdistance="0.005" altunitdist="inch" altunit="inch"/>
 <layers>
 <layer number="1" name="Top" color="4" fill="1" visible="yes" active="yes"/>
@@
 <wire x1="15.875" y1="10.795" x2="15.875" y2="21.463" width="0.3048" layer="1"/>
 <wire x1="34.036" y1="11.176" x2="34.29" y2="10.922" width="0.3048" layer="16"/>
-<contactref element="BM2" pad="VDD"/>
-<contactref element="BM2" pad="SS0"/>
 <wire x1="34.036" y1="11.176" x2="19.812" y2="25.4" width="0.3048" layer="16"/>
-<wire x1="38.2778" y1="10.0584" x2="38.2778" y2="7.8232" width="0.3048" layer="16"/>
-<wire x1="38.2778" y1="7.8232" x2="38.1" y2="7.62" width="0.3048" layer="16"/>
-<wire x1="38.2778" y1="10.0584" x2="38.1" y2="10.16" width="0.3048" layer="16"/>
-<wire x1="38.1" y1="10.16" x2="35.052" y2="10.16" width="0.3048" layer="16"/>
 <wire x1="35.052" y1="10.16" x2="34.036" y2="11.176" width="0.3048" layer="16"/>
+<contactref element="BM2" pad="VIN"/>
+<wire x1="38.1" y1="5.08" x2="36.83" y2="5.08" width="0.3048" layer="16"/>
+<wire x1="36.83" y1="5.08" x2="35.052" y2="6.858" width="0.3048" layer="16"/>
+<wire x1="35.052" y1="6.858" x2="35.052" y2="10.16" width="0.3048" layer="16"/>
 </signal>
 <signal name="P.TXD">
@@
 <wire x1="26.67" y1="25.4" x2="22.312" y2="25.4" width="0.3048" layer="16"/>
 </signal>
+<signal name="N$5">
+<contactref element="BM2" pad="VDD"/>
+<contactref element="BM2" pad="SS0"/>
+<wire x1="38.2778" y1="10.0584" x2="38.2778" y2="7.8232" width="0.3048" layer="16"/>
+<wire x1="38.2778" y1="7.8232" x2="38.1" y2="7.62" width="0.3048" layer="16"/>
+<wire x1="38.2778" y1="10.0584" x2="38.1" y2="10.16" width="0.3048" layer="16"/>
+</signal>
 </signals>
