File: LBriduino.sch (EAGLE design)
At the start: 12 parts, among them J1 105017-0001

Commit message: minor re-wireing, updated pic, specified usb connector in description
Connections:
- net GND: now also U$1.GND@3
Changed lines of the file:
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@@
 <part name="PROG" library="pinhead" library_urn="urn:adsk.eagle:library:325" deviceset="PINHD-1X4" device="" package3d_urn="urn:adsk.eagle:package:22407/2"/>
 <part name="BAT" library="pinhead" library_urn="urn:adsk.eagle:library:325" deviceset="PINHD-1X2" device="" package3d_urn="urn:adsk.eagle:package:22435/2"/>
+<part name="GND9" library="supply1" deviceset="GND" device=""/>
 </parts>
 <sheets>
@@
 <instance part="PROG" gate="A" x="127" y="15.24"/>
 <instance part="BAT" gate="G$1" x="127" y="40.64"/>
+<instance part="GND9" gate="1" x="33.02" y="17.78"/>
 </instances>
 <busses>
@@
 <label x="109.22" y="43.18" size="1.778" layer="95" rot="R180" xref="yes"/>
 </segment>
+<segment>
+<pinref part="U$1" gate="G$1" pin="GND@3"/>
+<wire x1="27.94" y1="15.24" x2="27.94" y2="22.86" width="0.1524" layer="91"/>
+<wire x1="27.94" y1="22.86" x2="33.02" y2="22.86" width="0.1524" layer="91"/>
+<pinref part="GND9" gate="1" pin="GND"/>
+<wire x1="33.02" y1="22.86" x2="33.02" y2="20.32" width="0.1524" layer="91"/>
+</segment>
 </net>

Commit message: changed BM019 voltage input from VIN to VDD, added testing points for ampere meter in off-mode
Parts:
- added C3: 100nF, resistor:C-EUC0603
- C1, C2: value 4.7µ -> 4.7µF
Connections:
- net N$3 renamed SCK
- net N$5 renamed MOSI
- net N$7 renamed MISO
- net N$8 renamed SS
- net N$9 renamed IRQ
- removed net N$10: BM2.SS0, BM2.VDD
- new net N$3: C3.2, PROG.4
- new net TEST: S1.3
- net P.RESET: now also C3.1; no longer PROG.4
- net SWITCH: now also BM2.SS0, BM2.VDD; no longer BM2.VIN
Changed lines of the file:
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@@
 <parts>
 <part name="U$1" library="RFD22301-11.25.13" deviceset="RFD22301" device=""/>
-<part name="C1" library="resistor" deviceset="C-EU" device="C0603" value="4.7µ"/>
-<part name="C2" library="resistor" deviceset="C-EU" device="C0603" value="4.7µ"/>
+<part name="C1" library="resistor" deviceset="C-EU" device="C0603" value="4.7µF"/>
+<part name="C2" library="resistor" deviceset="C-EU" device="C0603" value="4.7µF"/>
 <part name="R1" library="resistor" deviceset="R-EU_" device="R0603" value="331"/>
 <part name="LED1" library="led" deviceset="LED" device="CHIP-LED0603"/>
@@
 <part name="BAT" library="pinhead" library_urn="urn:adsk.eagle:library:325" deviceset="PINHD-1X2" device="" package3d_urn="urn:adsk.eagle:package:22435/2"/>
 <part name="GND9" library="supply1" deviceset="GND" device=""/>
+<part name="C3" library="resistor" deviceset="C-EU" device="C0603" value="100nF"/>
 </parts>
 <sheets>
@@
 <instance part="BAT" gate="G$1" x="127" y="40.64"/>
 <instance part="GND9" gate="1" x="33.02" y="17.78"/>
+<instance part="C3" gate="G$1" x="111.76" y="5.08" rot="R90"/>
 </instances>
 <busses>
@@
 <wire x1="71.12" y1="60.96" x2="71.12" y2="66.04" width="0.1524" layer="91"/>
 <pinref part="S1" gate="G$1" pin="1"/>
-<wire x1="71.12" y1="60.96" x2="83.82" y2="60.96" width="0.1524" layer="91"/>
+<wire x1="71.12" y1="60.96" x2="76.2" y2="60.96" width="0.1524" layer="91"/>
+<wire x1="78.74" y1="60.96" x2="83.82" y2="60.96" width="0.1524" layer="91"/>
 <wire x1="86.36" y1="60.96" x2="83.82" y2="60.96" width="0.1524" layer="91"/>
 <junction x="71.12" y="60.96"/>
+<wire x1="76.2" y1="60.96" x2="78.74" y2="60.96" width="0.1524" layer="91"/>
+<wire x1="78.74" y1="60.96" x2="78.74" y2="78.74" width="0.1524" layer="91"/>
 </segment>
 <segment>
@@
 </segment>
 </net>
-<net name="N$3" class="0">
+<net name="SCK" class="0">
 <segment>
 <pinref part="U$1" gate="G$1" pin="P0.04/AIN5"/>
@@
 </segment>
 </net>
-<net name="N$5" class="0">
+<net name="MOSI" class="0">
 <segment>
 <pinref part="U$1" gate="G$1" pin="P0.05/AIN6"/>
@@
 </segment>
 </net>
-<net name="N$7" class="0">
+<net name="MISO" class="0">
 <segment>
 <pinref part="U$1" gate="G$1" pin="P0.03/AIN4"/>
@@
 </segment>
 </net>
-<net name="N$8" class="0">
+<net name="SS" class="0">
 <segment>
 <pinref part="U$1" gate="G$1" pin="P0.06/AIN7"/>
@@
 </segment>
 </net>
-<net name="N$9" class="0">
+<net name="IRQ" class="0">
 <segment>
 <pinref part="U$1" gate="G$1" pin="P0.02/AIN3"/>
@@
 </segment>
 </net>
-<net name="N$10" class="0">
-<segment>
+<net name="SWITCH" class="0">
+<segment>
+<label x="53.34" y="0" size="1.778" layer="95" rot="MR0" xref="yes"/>
 <pinref part="BM2" gate="G$1" pin="VDD"/>
 <pinref part="BM2" gate="G$1" pin="SS0"/>
 <wire x1="58.42" y1="2.54" x2="58.42" y2="5.08" width="0.1524" layer="91"/>
-</segment>
-</net>
-<net name="SWITCH" class="0">
-<segment>
-<pinref part="BM2" gate="G$1" pin="VIN"/>
-<wire x1="53.34" y1="0" x2="58.42" y2="0" width="0.1524" layer="91"/>
-<label x="53.34" y="0" size="1.778" layer="95" rot="MR0" xref="yes"/>
+<wire x1="58.42" y1="2.54" x2="53.34" y2="2.54" width="0.1524" layer="91"/>
+<junction x="58.42" y="2.54"/>
+<wire x1="53.34" y1="2.54" x2="53.34" y2="0" width="0.1524" layer="91"/>
 </segment>
 <segment>
@@
 </segment>
 <segment>
+<pinref part="C3" gate="G$1" pin="1"/>
+<wire x1="109.22" y1="5.08" x2="104.14" y2="5.08" width="0.1524" layer="91"/>
+<label x="104.14" y="5.08" size="1.778" layer="95" rot="R180" xref="yes"/>
+</segment>
+</net>
+<net name="N$3" class="0">
+<segment>
 <pinref part="PROG" gate="A" pin="4"/>
-<wire x1="124.46" y1="12.7" x2="109.22" y2="12.7" width="0.1524" layer="91"/>
-<label x="109.22" y="12.7" size="1.778" layer="95" rot="R180" xref="yes"/>
-</segment>
-</net>
+<wire x1="124.46" y1="12.7" x2="119.38" y2="12.7" width="0.1524" layer="91"/>
+<wire x1="119.38" y1="12.7" x2="119.38" y2="5.08" width="0.1524" layer="91"/>
+<pinref part="C3" gate="G$1" pin="2"/>
+<wire x1="119.38" y1="5.08" x2="116.84" y2="5.08" width="0.1524" layer="91"/>
+</segment>
+</net>
+<net name="TEST" class="0">
+<segment>
+<pinref part="S1" gate="G$1" pin="3"/>
+<wire x1="83.82" y1="66.04" x2="83.82" y2="78.74" width="0.1524" layer="91"/>
+<wire x1="83.82" y1="78.74" x2="81.28" y2="78.74" width="0.1524" layer="91"/>
+</segment>
+</net>

Commit message: redesign: missing ground bugfix, charging-IC-cooling, bluetooth-area copper-free
Connections:
- removed net N$4: C1.2, C2.1
- net GND: now also C1.2, C2.1
- net P.RXD: now also PROG.2; no longer PROG.3
- net P.TXD: now also PROG.3; no longer PROG.2
Other:
- moved on the sheet: J1
Changed lines of the file:
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@@
 <?xml version="1.0" encoding="utf-8"?>
 <!DOCTYPE eagle SYSTEM "eagle.dtd">
-<eagle version="8.4.3">
+<eagle version="8.5.2">
 <drawing>
 <settings>
@@
 <part name="GND2" library="supply1" deviceset="GND" device=""/>
 <part name="P+2" library="supply1" library_urn="urn:adsk.eagle:library:371" deviceset="VCC" device=""/>
-<part name="J1" library="105017-0001" deviceset="105017-0001" device=""/>
 <part name="GND3" library="supply1" deviceset="GND" device=""/>
 <part name="BM2" library="Solutions Cubed" deviceset="BM019" device=""/>
@@
 <part name="GND9" library="supply1" deviceset="GND" device=""/>
 <part name="C3" library="resistor" deviceset="C-EU" device="C0603" value="100nF"/>
+<part name="GND10" library="supply1" deviceset="GND" device=""/>
+<part name="J1" library="105017-0001" deviceset="105017-0001" device=""/>
 </parts>
 <sheets>
@@
 <instance part="GND2" gate="1" x="58.42" y="48.26"/>
 <instance part="P+2" gate="VCC" x="71.12" y="68.58"/>
-<instance part="J1" gate="G$1" x="-22.86" y="66.04"/>
 <instance part="GND3" gate="1" x="-7.62" y="60.96"/>
 <instance part="BM2" gate="G$1" x="88.9" y="-2.54"/>
@@
 <instance part="GND9" gate="1" x="33.02" y="17.78"/>
 <instance part="C3" gate="G$1" x="111.76" y="5.08" rot="R90"/>
+<instance part="GND10" gate="1" x="35.56" y="68.58"/>
+<instance part="J1" gate="G$1" x="-25.4" y="66.04"/>
 </instances>
 <busses>
@@
 <pinref part="U$2" gate="G$1" pin="STAT"/>
 <wire x1="30.48" y1="53.34" x2="33.02" y2="53.34" width="0.1524" layer="91"/>
-</segment>
-</net>
-<net name="N$4" class="0">
-<segment>
-<pinref part="C2" gate="G$1" pin="1"/>
-<pinref part="C1" gate="G$1" pin="2"/>
-<wire x1="38.1" y1="73.66" x2="33.02" y2="73.66" width="0.1524" layer="91"/>
 </segment>
 </net>
@@
 <wire x1="-2.54" y1="73.66" x2="2.54" y2="73.66" width="0.1524" layer="91"/>
 <junction x="10.16" y="73.66"/>
-<pinref part="J1" gate="G$1" pin="VDD"/>
 <wire x1="2.54" y1="73.66" x2="10.16" y2="73.66" width="0.1524" layer="91"/>
-<wire x1="-10.16" y1="68.58" x2="2.54" y2="68.58" width="0.1524" layer="91"/>
+<wire x1="-12.7" y1="68.58" x2="2.54" y2="68.58" width="0.1524" layer="91"/>
 <wire x1="2.54" y1="68.58" x2="2.54" y2="73.66" width="0.1524" layer="91"/>
 <junction x="2.54" y="73.66"/>
+<pinref part="J1" gate="G$1" pin="VDD"/>
 </segment>
 </net>
@@
 </segment>
 <segment>
+<pinref part="GND3" gate="1" pin="GND"/>
+<wire x1="-12.7" y1="63.5" x2="-7.62" y2="63.5" width="0.1524" layer="91"/>
 <pinref part="J1" gate="G$1" pin="GND"/>
-<pinref part="GND3" gate="1" pin="GND"/>
-<wire x1="-10.16" y1="63.5" x2="-7.62" y2="63.5" width="0.1524" layer="91"/>
 </segment>
 <segment>
@@
 <pinref part="GND9" gate="1" pin="GND"/>
 <wire x1="33.02" y1="22.86" x2="33.02" y2="20.32" width="0.1524" layer="91"/>
+</segment>
+<segment>
+<pinref part="C2" gate="G$1" pin="1"/>
+<pinref part="C1" gate="G$1" pin="2"/>
+<wire x1="38.1" y1="73.66" x2="35.56" y2="73.66" width="0.1524" layer="91"/>
+<pinref part="GND10" gate="1" pin="GND"/>
+<wire x1="35.56" y1="73.66" x2="33.02" y2="73.66" width="0.1524" layer="91"/>
+<wire x1="35.56" y1="71.12" x2="35.56" y2="73.66" width="0.1524" layer="91"/>
+<junction x="35.56" y="73.66"/>
 </segment>
 </net>
@@
 </segment>
 <segment>
-<pinref part="PROG" gate="A" pin="2"/>
-<wire x1="124.46" y1="17.78" x2="109.22" y2="17.78" width="0.1524" layer="91"/>
-<label x="109.22" y="17.78" size="1.778" layer="95" rot="R180" xref="yes"/>
+<pinref part="PROG" gate="A" pin="3"/>
+<wire x1="124.46" y1="15.24" x2="99.06" y2="15.24" width="0.1524" layer="91"/>
+<label x="99.06" y="15.24" size="1.778" layer="95" rot="R180" xref="yes"/>
 </segment>
 </net>
@@
 </segment>
 <segment>
-<pinref part="PROG" gate="A" pin="3"/>
-<wire x1="124.46" y1="15.24" x2="99.06" y2="15.24" width="0.1524" layer="91"/>
-<label x="99.06" y="15.24" size="1.778" layer="95" rot="R180" xref="yes"/>
-</segment>
-</net>
+<pinref part="PROG" gate="A" pin="2"/>
+<wire x1="124.46" y1="17.78" x2="109.22" y2="17.78" width="0.1524" layer="91"/>
+<label x="109.22" y="17.78" size="1.778" layer="95" rot="R180" xref="yes"/>
+</segment>
+</net>
